File: PCB/PCB.kicad_sch (KiCad schematic)
At the start: 22 parts, among them J1 Servo_Conn_1, J10 Conn_01x04_Pin, J11 UBEC_Pow_In, J12 Spare_GPIO_Conn, J2 Servo_Conn_2, J3 Servo_Conn_3, J4 Servo_Conn_4, J5 Servo_Conn_5, J6 Servo_Conn_6, J7 Mot1_Conn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

Commit message: update pcb layout
Parts:
- J10, J9: footprint Connector_PinHeader_2.54mm:PinHeader_1x04_P2.54mm_Vertical -> Connector_PinHeader_2.54mm:PinHeader_2x02_P2.54mm_Vertical
Connections:
- net INA1: now also MOT_DRV_Conn1.6 (Pin_6); no longer MOT_DRV_Conn1.5 (Pin_5)
- net INA2: now also MOT_DRV_Conn1.5 (Pin_5); no longer MOT_DRV_Conn1.6 (Pin_6)
- net INB1: now also MOT_DRV_Conn1.8 (Pin_8); no longer MOT_DRV_Conn1.7 (Pin_7)
- net INB2: now also MOT_DRV_Conn1.7 (Pin_7); no longer MOT_DRV_Conn1.8 (Pin_8)
- net PWM1: now also MOT_DRV_Conn1.4 (Pin_4); no longer MOT_DRV_Conn1.3 (Pin_3)
- net PWM2: now also MOT_DRV_Conn1.3 (Pin_3); no longer MOT_DRV_Conn1.4 (Pin_4)
Changed lines of the file:
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@@
 	)
 	(label "INB1"
-		(at 189.23 50.8 0)
-		(effects
-			(font
-				(size 1.27 1.27)
-			)
-			(justify left bottom)
+		(at 224.79 50.8 180)
+		(effects
+			(font
+				(size 1.27 1.27)
+			)
+			(justify right bottom)
 		)
 	)
@@
 	)
 	(label "PWM2"
-		(at 224.79 45.72 180)
-		(effects
-			(font
-				(size 1.27 1.27)
-			)
-			(justify right bottom)
+		(at 189.23 45.72 0)
+		(effects
+			(font
+				(size 1.27 1.27)
+			)
+			(justify left bottom)
 		)
 	)
@@
 	)
 	(label "INA1"
-		(at 189.23 48.26 0)
-		(effects
-			(font
-				(size 1.27 1.27)
-			)
-			(justify left bottom)
+		(at 224.79 48.26 180)
+		(effects
+			(font
+				(size 1.27 1.27)
+			)
+			(justify right bottom)
 		)
 	)
@@
 	)
 	(label "INA2"
-		(at 224.79 48.26 180)
-		(effects
-			(font
-				(size 1.27 1.27)
-			)
-			(justify right bottom)
+		(at 189.23 48.26 0)
+		(effects
+			(font
+				(size 1.27 1.27)
+			)
+			(justify left bottom)
 		)
 	)
@@
 	)
 	(label "PWM1"
-		(at 189.23 45.72 0)
-		(effects
-			(font
-				(size 1.27 1.27)
-			)
-			(justify left bottom)
+		(at 224.79 45.72 180)
+		(effects
+			(font
+				(size 1.27 1.27)
+			)
+			(justify right bottom)
 		)
 	)
@@
 	)
 	(label "INB2"
-		(at 224.79 50.8 180)
-		(effects
-			(font
-				(size 1.27 1.27)
-			)
-			(justify right bottom)
+		(at 189.23 50.8 0)
+		(effects
+			(font
+				(size 1.27 1.27)
+			)
+			(justify left bottom)
 		)
 	)
@@
 			)
 		)
-		(property "Footprint" "Connector_PinHeader_2.54mm:PinHeader_1x04_P2.54mm_Vertical"
+		(property "Footprint" "Connector_PinHeader_2.54mm:PinHeader_2x02_P2.54mm_Vertical"
 			(at 240.03 81.28 0)
 			(effects
@@
 			)
 		)
-		(property "Footprint" "Connector_PinHeader_2.54mm:PinHeader_1x04_P2.54mm_Vertical"
+		(property "Footprint" "Connector_PinHeader_2.54mm:PinHeader_2x02_P2.54mm_Vertical"
 			(at 153.67 81.28 0)
 			(effects

Commit message: wire up
Parts:
- H1, H2, H3, H4: footprint MountingHole:MountingHole_2.7mm_M2.5 -> MountingHole:MountingHole_2.7mm_M2.5_Pad_Via
Changed lines of the file:
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@@
 			)
 		)
-		(property "Footprint" "MountingHole:MountingHole_2.7mm_M2.5"
+		(property "Footprint" "MountingHole:MountingHole_2.7mm_M2.5_Pad_Via"
 			(at 163.83 165.1 0)
 			(effects
@@
 			)
 		)
-		(property "Footprint" "MountingHole:MountingHole_2.7mm_M2.5"
+		(property "Footprint" "MountingHole:MountingHole_2.7mm_M2.5_Pad_Via"
 			(at 134.62 165.1 0)
 			(effects
@@
 			)
 		)
-		(property "Footprint" "MountingHole:MountingHole_2.7mm_M2.5"
+		(property "Footprint" "MountingHole:MountingHole_2.7mm_M2.5_Pad_Via"
 			(at 134.62 154.94 0)
 			(effects
@@
 			)
 		)
-		(property "Footprint" "MountingHole:MountingHole_2.7mm_M2.5"
+		(property "Footprint" "MountingHole:MountingHole_2.7mm_M2.5_Pad_Via"
 			(at 163.83 154.94 0)
 			(effects
